Commit message: feat: add T1 29dof whole body tracking support

File: src/holosoma_retargeting/holosoma_retargeting/models/largebox/largebox.urdf (robot description, URDF)
Before this commit: robot largebox, 1 links, 0 joints
Links:
- removed link largebox_link
- added link baseLink; collision mesh filename=objects/largebox/largebox.obj scale=1.0 1.0 1.0; visual mesh filename=objects/largebox/largebox.obj scale=1.0 1.0 1.0
